File: 16_8_2020project/16_8_2020project.kicad_pcb (KiCad board)
At the start: 2 copper layers, 51.2 x 26.2 mm, 12 parts, among them J1 PJ-102AH, J2 Conn_02x02_Odd_Even, J3 Conn_02x02_Odd_Even, U1 AZ1117CH-3.3TRG1, U2 AZ1117CH-5.0TRG1

Commit message: Add files via upload
build 2
Routing:
- net GND: track 6.23 -> 51.8 mm, vias 27 -> 34
- net Net-(D1-Pad2): track 7.00 -> 14.1 mm
- net Net-(C3-Pad1): track 82.2 -> 83.9 mm
Other:
- board size 51.2 x 26.2 mm -> 52.5 x 27 mm
- rule pad_to_mask_clearance: 0.051 -> 0.0762
- board text added: "+"
- board text added: "-"
- board text added: "3.3v"
- board text added: "5v"
