File: 16_8_2020project/16_8_2020project.sch (KiCad schematic (older format))
At the start: 11 parts, among them J1 PJ-102AH, J2 Conn_02x02_Odd_Even, J3 Conn_02x02_Odd_Even, U1 AZ1117CH-3.3TRG1, U2 AZ1117CH-5.0TRG1

Commit message: Add files via upload
Other:
- note added: "MIT License\n\nCopyright (c) 2020 ShaikMoosa\n\nPermission is hereby granted, free of charge, to any person obtaining a copy\nof this software and associated documentation files (the "Software"), to deal\nin the Software without restriction, including without limitation the rights\nto use, copy, modify, merge, publish, distribute, sublicense, and/or sell\ncopies of the Software, and to permit per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"
Changed lines of the file:
@@
 Wire Wire Line
 	6350 3800 7300 3800
+Text Notes 6350 7250 0    14   ~ 0
+MIT License\n\nCopyright (c) 2020 ShaikMoosa\n\nPermission is hereby granted, free of charge, to any person obtaining a copy\nof this software and associated documentation files (the "Software"), to deal\nin the Software without restriction, including without limitation the rights\nto use, copy, modify, merge, publish, distribute, sublicense, and/or sell\ncopies of the Software, and to permit persons to whom the Software is\nfurnished to do so, subject to the following conditions:\n\nThe above copyright notice and this permission notice shall be included in all\ncopies or substantial portions of the Software.\n\nTHE SOFTWARE IS PROVIDED "AS IS", WITHOUT WARRANTY OF ANY KIND, EXPRESS OR\nIMPLIED, INCLUDING BUT NOT LIMITED TO THE WARRANTIES OF MERCHANTABILITY,\nFITNESS FOR A PARTICULAR PURPOSE AND NONINFRINGEMENT. IN NO EVENT SHALL THE\nAUTHORS OR COPYRIGHT HOLDERS BE LIABLE FOR ANY CLAIM, DAMAGES OR OTHER\nLIABILITY, WHETHER IN AN ACTION OF CONTRACT, TORT OR OTHERWISE, ARISING FROM,\nOUT OF OR IN CONNECTION WITH THE SOFTWARE OR THE USE OR OTHER DEALINGS IN THE\nSOFTWARE.
 $EndSCHEMATC
